Commit message: multi-UAV

File: rotors_description/urdf/component_snippets.xacro (robot description, xacro)
@@ -242,5 +242,5 @@
         <commandMotorSpeedSubTopic>command/motor_speed</commandMotorSpeedSubTopic>
         <imuSubTopic>${imu_sub_topic}</imuSubTopic>
-        <motorSpeedCommandPubTopic>gazebo/command/motor_speed</motorSpeedCommandPubTopic>
+        <motorSpeedCommandPubTopic>gazebo/command/motor_speed_switch</motorSpeedCommandPubTopic>
       </plugin>
     </gazebo>
@@ -884,5 +884,5 @@
       imu_sub_topic="${imu_sub_topic}"
       mavlink_pub_topic="/mavlink/to"
-      motors_speeds_pub_topic="gazebo/command/motor_speed"
+      motors_speeds_pub_topic="gazebo/command/motor_speed_switch"
       gps_update_freq="5.0"
       rotor_count="${rotor_count}"

File: rotors_description/urdf/firefly.xacro (robot description, xacro)
@@ -47,8 +47,38 @@
   </xacro:property>
   <!-- Included URDF Files -->
-  <xacro:include filename="$(find rotors_description)/urdf/multirotor_base.xacro" />
+  <xacro:include filename="$(find rotors_description)/urdf/final.xacro"/>
   <!-- Instantiate multirotor_base_macro once -->
   <xacro:multirotor_base_macro
     robot_namespace="${namespace}"
+    mass="${mass}"
+    body_width="${body_width}"
+    body_height="${body_height}"
+    use_mesh_file="${use_mesh_file}"
+    mesh_file="${mesh_file}"
+    >
+    <xacro:insert_block name="body_inertia" />
+  </xacro:multirotor_base_macro>
+  <xacro:multirotor_base_macro
+    robot_namespace="firefly2"
+    mass="${mass}"
+    body_width="${body_width}"
+    body_height="${body_height}"
+    use_mesh_file="${use_mesh_file}"
+    mesh_file="${mesh_file}"
+    >
+    <xacro:insert_block name="body_inertia" />
+  </xacro:multirotor_base_macro>
+  <xacro:multirotor_base_macro
+    robot_namespace="firefly3"
+    mass="${mass}"
+    body_width="${body_width}"
+    body_height="${body_height}"
+    use_mesh_file="${use_mesh_file}"
+    mesh_file="${mesh_file}"
+    >
+    <xacro:insert_block name="body_inertia" />
+  </xacro:multirotor_base_macro>
+  <xacro:multirotor_base_macro
+    robot_namespace="firefly4"
     mass="${mass}"
     body_width="${body_width}"
@@ -184,3 +214,387 @@
     <xacro:insert_block name="rotor_inertia" />
   </xacro:vertical_rotor>
+<!--firefly2-->
+<!-- Instantiate rotors -->
+<xacro:vertical_rotor
+  robot_namespace="firefly2"
+  suffix="front_left"
+  direction="ccw"
+  motor_constant="${motor_constant}"
+  moment_constant="${moment_constant}"
+  parent="firefly2/base_link"
+  mass_rotor="${mass_rotor}"
+  radius_rotor="${radius_rotor}"
+  time_constant_up="${time_constant_up}"
+  time_constant_down="${time_constant_down}"
+  max_rot_velocity="${max_rot_velocity}"
+  motor_number="0"
+  rotor_drag_coefficient="${rotor_drag_coefficient}"
+  rolling_moment_coefficient="${rolling_moment_coefficient}"
+  color="Red"
+  use_own_mesh="false"
+  mesh="">
+  <origin xyz="${cos30*arm_length} ${sin30*arm_length} ${rotor_offset_top}" rpy="0 0 0" />
+  <xacro:insert_block name="rotor_inertia" />
+</xacro:vertical_rotor>
+<xacro:vertical_rotor
+  robot_namespace="firefly2"
+  suffix="left"
+  direction="cw"
+  motor_constant="${motor_constant}"
+  moment_constant="${moment_constant}"
+  parent="firefly2/base_link"
+  mass_rotor="${mass_rotor}"
+  radius_rotor="${radius_rotor}"
+  time_constant_up="${time_constant_up}"
+  time_constant_down="${time_constant_down}"
+  max_rot_velocity="${max_rot_velocity}"
+  motor_number="1"
+  rotor_drag_coefficient="${rotor_drag_coefficient}"
+  rolling_moment_coefficient="${rolling_moment_coefficient}"
+  color="Blue"
+  use_own_mesh="false"
+  mesh="">
+  <origin xyz="0 ${arm_length} ${rotor_offset_top}" rpy="0 0 0" />
+  <xacro:insert_block name="rotor_inertia" />
+</xacro:vertical_rotor>
+<xacro:vertical_rotor robot_namespace="firefly2"
+  suffix="back_left"
+  direction="ccw"
+  motor_constant="${motor_constant}"
+  moment_constant="${moment_constant}"
+  parent="firefly2/base_link"
+  mass_rotor="${mass_rotor}"
+  radius_rotor="${radius_rotor}"
+  time_constant_up="${time_constant_up}"
+  time_constant_down="${time_constant_down}"
+  max_rot_velocity="${max_rot_velocity}"
+  motor_number="2"
+  rotor_drag_coefficient="${rotor_drag_coefficient}"
+  rolling_moment_coefficient="${rolling_moment_coefficient}"
+  color="Blue"
+  use_own_mesh="false"
+  mesh="">
+  <origin xyz="-${cos30*arm_length} ${sin30*arm_length} ${rotor_offset_top}" rpy="0 0 0" />
+  <xacro:insert_block name="rotor_inertia" />
+</xacro:vertical_rotor>
+<xacro:vertical_rotor robot_namespace="firefly2"
+  suffix="back_right"
+  direction="cw"
+  motor_constant="${motor_constant}"
+  moment_constant="${moment_constant}"
+  parent="firefly2/base_link"
+  mass_rotor="${mass_rotor}"
+  radius_rotor="${radius_rotor}"
+  time_constant_up="${time_constant_up}"
+  time_constant_down="${time_constant_down}"
+  max_rot_velocity="${max_rot_velocity}"
+  motor_number="3"
+  rotor_drag_coefficient="${rotor_drag_coefficient}"
+  rolling_moment_coefficient="${rolling_moment_coefficient}"
+  color="Blue"
+  use_own_mesh="false"
+  mesh="">
+  <origin xyz="-${cos30*arm_length} -${sin30*arm_length} ${rotor_offset_top}" rpy="0 0 0" />
+  <xacro:insert_block name="rotor_inertia" />
+</xacro:vertical_rotor>
+<xacro:vertical_rotor
+  robot_namespace="firefly2"
+  suffix="right"
+  direction="ccw"
+  motor_constant="${motor_constant}"
+  moment_constant="${moment_constant}"
+  parent="firefly2/base_link"
+  mass_rotor="${mass_rotor}"
+  radius_rotor="${radius_rotor}"
+  time_constant_up="${time_constant_up}"
+  time_constant_down="${time_constant_down}"
+  max_rot_velocity="${max_rot_velocity}"
+  motor_number="4"
+  rotor_drag_coefficient="${rotor_drag_coefficient}"
+  rolling_moment_coefficient="${rolling_moment_coefficient}"
+  color="Blue"
+  use_own_mesh="false"
+  mesh="">
+  <origin xyz="0 -${arm_length} ${rotor_offset_top}" rpy="0 0 0" />
+  <xacro:insert_block name="rotor_inertia" />
+</xacro:vertical_rotor>
+<xacro:vertical_rotor
+  robot_namespace="firefly2"
+  suffix="front_right"
+  direction="cw"
+  motor_constant="${motor_constant}"
+  moment_constant="${moment_constant}"
+  parent="firefly2/base_link"
+  mass_rotor="${mass_rotor}"
+  radius_rotor="${radius_rotor}"
+  time_constant_up="${time_constant_up}"
+  time_constant_down="${time_constant_down}"
+  max_rot_velocity="${max_rot_velocity}"
+  motor_number="5"
+  rotor_drag_coefficient="${rotor_drag_coefficient}"
+  rolling_moment_coefficient="${rolling_moment_coefficient}"
+  color="Red"
+  use_own_mesh="false"
+  mesh="">
+  <origin xyz="${cos30*arm_length} -${sin30*arm_length} ${rotor_offset_top}" rpy="0 0 0" />
+  <xacro:insert_block name="rotor_inertia" />
+</xacro:vertical_rotor>
+<!--firefly3-->
+<!-- Instantiate rotors -->
+<xacro:vertical_rotor
+  robot_namespace="firefly3"
+  suffix="front_left"
+  direction="ccw"
+  motor_constant="${motor_constant}"
+  moment_constant="${moment_constant}"
+  parent="firefly3/base_link"
+  mass_rotor="${mass_rotor}"
+  radius_rotor="${radius_rotor}"
+  time_constant_up="${time_constant_up}"
+  time_constant_down="${time_constant_down}"
+  max_rot_velocity="${max_rot_velocity}"
+  motor_number="0"
+  rotor_drag_coefficient="${rotor_drag_coefficient}"
+  rolling_moment_coefficient="${rolling_moment_coefficient}"
+  color="Red"
+  use_own_mesh="false"
+  mesh="">
+  <origin xyz="${cos30*arm_length} ${sin30*arm_length} ${rotor_offset_top}" rpy="0 0 0" />
+  <xacro:insert_block name="rotor_inertia" />
+</xacro:vertical_rotor>
+<xacro:vertical_rotor
+  robot_namespace="firefly3"
+  suffix="left"
+  direction="cw"
+  motor_constant="${motor_constant}"
+  moment_constant="${moment_constant}"
+  parent="firefly3/base_link"
+  mass_rotor="${mass_rotor}"
+  radius_rotor="${radius_rotor}"
+  time_constant_up="${time_constant_up}"
+  time_constant_down="${time_constant_down}"
+  max_rot_velocity="${max_rot_velocity}"
+  motor_number="1"
+  rotor_drag_coefficient="${rotor_drag_coefficient}"
+  rolling_moment_coefficient="${rolling_moment_coefficient}"
+  color="Blue"
+  use_own_mesh="false"
+  mesh="">
+  <origin xyz="0 ${arm_length} ${rotor_offset_top}" rpy="0 0 0" />
+  <xacro:insert_block name="rotor_inertia" />
+</xacro:vertical_rotor>
+<xacro:vertical_rotor robot_namespace="firefly3"
+  suffix="back_left"
+  direction="ccw"
+  motor_constant="${motor_constant}"
+  moment_constant="${moment_constant}"
+  parent="firefly3/base_link"
+  mass_rotor="${mass_rotor}"
+  radius_rotor="${radius_rotor}"
+  time_constant_up="${time_constant_up}"
+  time_constant_down="${time_constant_down}"
+  max_rot_velocity="${max_rot_velocity}"
+  motor_number="2"
+  rotor_drag_coefficient="${rotor_drag_coefficient}"
+  rolling_moment_coefficient="${rolling_moment_coefficient}"
+  color="Blue"
+  use_own_mesh="false"
+  mesh="">
+  <origin xyz="-${cos30*arm_length} ${sin30*arm_length} ${rotor_offset_top}" rpy="0 0 0" />
+  <xacro:insert_block name="rotor_inertia" />
+</xacro:vertical_rotor>
+<xacro:vertical_rotor robot_namespace="firefly3"
+  suffix="back_right"
+  direction="cw"
+  motor_constant="${motor_constant}"
+  moment_constant="${moment_constant}"
+  parent="firefly3/base_link"
+  mass_rotor="${mass_rotor}"
+  radius_rotor="${radius_rotor}"
+  time_constant_up="${time_constant_up}"
+  time_constant_down="${time_constant_down}"
+  max_rot_velocity="${max_rot_velocity}"
+  motor_number="3"
+  rotor_drag_coefficient="${rotor_drag_coefficient}"
+  rolling_moment_coefficient="${rolling_moment_coefficient}"
+  color="Blue"
+  use_own_mesh="false"
+  mesh="">
+  <origin xyz="-${cos30*arm_length} -${sin30*arm_length} ${rotor_offset_top}" rpy="0 0 0" />
+  <xacro:insert_block name="rotor_inertia" />
+</xacro:vertical_rotor>
+<xacro:vertical_rotor
+  robot_namespace="firefly3"
+  suffix="right"
+  direction="ccw"
+  motor_constant="${motor_constant}"
+  moment_constant="${moment_constant}"
+  parent="firefly3/base_link"
+  mass_rotor="${mass_rotor}"
+  radius_rotor="${radius_rotor}"
+  time_constant_up="${time_constant_up}"
+  time_constant_down="${time_constant_down}"
+  max_rot_velocity="${max_rot_velocity}"
+  motor_number="4"
+  rotor_drag_coefficient="${rotor_drag_coefficient}"
+  rolling_moment_coefficient="${rolling_moment_coefficient}"
+  color="Blue"
+  use_own_mesh="false"
+  mesh="">
+  <origin xyz="0 -${arm_length} ${rotor_offset_top}" rpy="0 0 0" />
+  <xacro:insert_block name="rotor_inertia" />
+</xacro:vertical_rotor>
+<xacro:vertical_rotor
+  robot_namespace="firefly3"
+  suffix="front_right"
+  direction="cw"
+  motor_constant="${motor_constant}"
+  moment_constant="${moment_constant}"
+  parent="firefly3/base_link"
+  mass_rotor="${mass_rotor}"
+  radius_rotor="${radius_rotor}"
+  time_constant_up="${time_constant_up}"
+  time_constant_down="${time_constant_down}"
+  max_rot_velocity="${max_rot_velocity}"
+  motor_number="5"
+  rotor_drag_coefficient="${rotor_drag_coefficient}"
+  rolling_moment_coefficient="${rolling_moment_coefficient}"
+  color="Red"
+  use_own_mesh="false"
+  mesh="">
+  <origin xyz="${cos30*arm_length} -${sin30*arm_length} ${rotor_offset_top}" rpy="0 0 0" />
+  <xacro:insert_block name="rotor_inertia" />
+</xacro:vertical_rotor>
+<!--firefly4-->
+<!-- Instantiate rotors -->
+<xacro:vertical_rotor
+  robot_namespace="firefly4"
+  suffix="front_left"
+  direction="ccw"
+  motor_constant="${motor_constant}"
+  moment_constant="${moment_constant}"
+  parent="firefly4/base_link"
+  mass_rotor="${mass_rotor}"
+  radius_rotor="${radius_rotor}"
+  time_constant_up="${time_constant_up}"
+  time_constant_down="${time_constant_down}"
+  max_rot_velocity="${max_rot_velocity}"
+  motor_number="0"
+  rotor_drag_coefficient="${rotor_drag_coefficient}"
+  rolling_moment_coefficient="${rolling_moment_coefficient}"
+  color="Red"
+  use_own_mesh="false"
+  mesh="">
+  <origin xyz="${cos30*arm_length} ${sin30*arm_length} ${rotor_offset_top}" rpy="0 0 0" />
+  <xacro:insert_block name="rotor_inertia" />
+</xacro:vertical_rotor>
+<xacro:vertical_rotor
+  robot_namespace="firefly4"
+  suffix="left"
+  direction="cw"
+  motor_constant="${motor_constant}"
+  moment_constant="${moment_constant}"
+  parent="firefly4/base_link"
+  mass_rotor="${mass_rotor}"
+  radius_rotor="${radius_rotor}"
+  time_constant_up="${time_constant_up}"
+  time_constant_down="${time_constant_down}"
+  max_rot_velocity="${max_rot_velocity}"
+  motor_number="1"
+  rotor_drag_coefficient="${rotor_drag_coefficient}"
+  rolling_moment_coefficient="${rolling_moment_coefficient}"
+  color="Blue"
+  use_own_mesh="false"
+  mesh="">
+  <origin xyz="0 ${arm_length} ${rotor_offset_top}" rpy="0 0 0" />
+  <xacro:insert_block name="rotor_inertia" />
+</xacro:vertical_rotor>
+<xacro:vertical_rotor robot_namespace="firefly4"
+  suffix="back_left"
+  direction="ccw"
+  motor_constant="${motor_constant}"
+  moment_constant="${moment_constant}"
+  parent="firefly4/base_link"
+  mass_rotor="${mass_rotor}"
+  radius_rotor="${radius_rotor}"
+  time_constant_up="${time_constant_up}"
+  time_constant_down="${time_constant_down}"
+  max_rot_velocity="${max_rot_velocity}"
+  motor_number="2"
+  rotor_drag_coefficient="${rotor_drag_coefficient}"
+  rolling_moment_coefficient="${rolling_moment_coefficient}"
+  color="Blue"
+  use_own_mesh="false"
+  mesh="">
+  <origin xyz="-${cos30*arm_length} ${sin30*arm_length} ${rotor_offset_top}" rpy="0 0 0" />
+  <xacro:insert_block name="rotor_inertia" />
+</xacro:vertical_rotor>
+<xacro:vertical_rotor robot_namespace="firefly4"
+  suffix="back_right"
+  direction="cw"
+  motor_constant="${motor_constant}"
+  moment_constant="${moment_constant}"
+  parent="firefly4/base_link"
+  mass_rotor="${mass_rotor}"
+  radius_rotor="${radius_rotor}"
+  time_constant_up="${time_constant_up}"
+  time_constant_down="${time_constant_down}"
+  max_rot_velocity="${max_rot_velocity}"
+  motor_number="3"
+  rotor_drag_coefficient="${rotor_drag_coefficient}"
+  rolling_moment_coefficient="${rolling_moment_coefficient}"
+  color="Blue"
+  use_own_mesh="false"
+  mesh="">
+  <origin xyz="-${cos30*arm_length} -${sin30*arm_length} ${rotor_offset_top}" rpy="0 0 0" />
+  <xacro:insert_block name="rotor_inertia" />
+</xacro:vertical_rotor>
+<xacro:vertical_rotor
+  robot_namespace="firefly4"
+  suffix="right"
+  direction="ccw"
+  motor_constant="${motor_constant}"
+  moment_constant="${moment_constant}"
+  parent="firefly4/base_link"
+  mass_rotor="${mass_rotor}"
+  radius_rotor="${radius_rotor}"
+  time_constant_up="${time_constant_up}"
+  time_constant_down="${time_constant_down}"
+  max_rot_velocity="${max_rot_velocity}"
+  motor_number="4"
+  rotor_drag_coefficient="${rotor_drag_coefficient}"
+  rolling_moment_coefficient="${rolling_moment_coefficient}"
+  color="Blue"
+  use_own_mesh="false"
+  mesh="">
+  <origin xyz="0 -${arm_length} ${rotor_offset_top}" rpy="0 0 0" />
+  <xacro:insert_block name="rotor_inertia" />
+</xacro:vertical_rotor>
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
File: rotors_description/urdf/single_base.xacro (robot description, xacro)
@@ -19,10 +19,7 @@
   <xacro:include filename="$(find rotors_description)/urdf/component_snippets.xacro" />
   <!-- Instantiate firefly "mechanics" -->
-  <xacro:include filename="$(find rotors_description)/urdf/firefly.xacro" />
+  <xacro:include filename="$(find rotors_description)/urdf/single.xacro" />
   <!-- Instantiate a controller. -->
   <xacro:controller_plugin_macro namespace="${namespace}" imu_sub_topic="imu" />
-  <xacro:controller_plugin_macro namespace="firefly2" imu_sub_topic="imu" />
-  <xacro:controller_plugin_macro namespace="firefly3" imu_sub_topic="imu" />
-  <xacro:controller_plugin_macro namespace="firefly4" imu_sub_topic="imu" />
   <!-- Instantiate a ROS message interface -->
   <!-- <xacro:ros_interface_plugin_macro namespace="${namespace}" />-->
@@ -30,18 +27,9 @@
     <!-- Instantiate mavlink telemetry interface. -->
     <xacro:default_mavlink_interface namespace="${namespace}" imu_sub_topic="imu" rotor_count="6" />
-    <xacro:default_mavlink_interface namespace="firefly2" imu_sub_topic="imu" rotor_count="6" />
-    <xacro:default_mavlink_interface namespace="firefly3" imu_sub_topic="imu" rotor_count="6" />
-    <xacro:default_mavlink_interface namespace="firefly4" imu_sub_topic="imu" rotor_count="6" />
   </xacro:if>
   <!-- Mount an ADIS16448 IMU. -->
   <xacro:default_imu namespace="${namespace}" parent_link="${namespace}/base_link" />
-  <xacro:default_imu namespace="firefly2" parent_link="firefly2/base_link" />
-  <xacro:default_imu namespace="firefly3" parent_link="firefly3/base_link" />
-  <xacro:default_imu namespace="firefly4" parent_link="firefly4/base_link" />
   <xacro:if value="$(arg enable_ground_truth)">
     <xacro:ground_truth_imu_and_odometry namespace="${namespace}" parent_link="${namespace}/base_link" />
-    <xacro:ground_truth_imu_and_odometry namespace="firefly2" parent_link="firefly2/base_link" />
-    <xacro:ground_truth_imu_and_odometry namespace="firefly3" parent_link="firefly3/base_link" />
-    <xacro:ground_truth_imu_and_odometry namespace="firefly4" parent_link="firefly4/base_link" />
   </xacro:if>
   <xacro:if value="$(arg enable_logging)">
